Commit message: changes

File: Manipulator/man_gazebo/urdf/6dof/full_manipulator.urdf.xacro (robot description, xacro)
@@ -1,4 +1,12 @@
 <?xml version="1.0"?>
-<robot xmlns:xacro="http://wiki.ros.org/xacro">
+<robot xmlns:xacro="http://wiki.ros.org/xacro" name="arm" >
+<!-- common stuff -->
+<xacro:include filename="$(find man_gazebo)/urdf/common.gazebo.xacro" />
+<link name="world" />
+  <joint name="world_joint" type="fixed">
+    <parent link="world" />
+    <child link = "base_link" />
+    <origin xyz="0 0 0" rpy="0.0 0.0 0.0" />
+  </joint>
   <xacro:include filename="$(find man_gazebo)/urdf/transmission.xacro" />
   <xacro:include filename="$(find man_gazebo)/urdf/gazebo.xacro" />
@@ -24,23 +32,5 @@
 </xacro:macro>
   <xacro:macro name="arm_robot" params="prefix ">
-    <xacro:property name="joint1_type" value="revolute" />
-	<xacro:property name="joint2_type" value="revolute" />
-	<xacro:property name="joint3_type" value="revolute" />
-	<xacro:property name="joint4_type" value="revolute" />
-	<xacro:property name="joint5_type" value="revolute" />
-	<xacro:property name="joint6_type" value="revolute" />
-	<xacro:property name="joint1_axe" value="0 0 1" />
-	<xacro:property name="joint2_axe" value="0 1 0" />
-	<xacro:property name="joint3_axe" value="0 1 0" />
-	<xacro:property name="joint4_axe" value="0 1 0" />
-	<xacro:property name="joint5_axe" value="0 1 0" />
-	<xacro:property name="joint6_axe" value="0 0 1" />
     <xacro:property name="base_length" value="0.25" />
-	<xacro:property name="link1_length" value="0.15" />
-	<xacro:property name="link2_length" value="0.5" />
-	<xacro:property name="link3_length" value="0.4" />
-	<xacro:property name="link4_length" value="0.07" />
-	<xacro:property name="link5_length" value="0.1" />
-	<xacro:property name="link6_length" value="0.02" />
     <!-- Inertia parameters -->
     <xacro:property name="base_mass" value="4.0" />
@@ -58,5 +48,5 @@
     <xacro:property name="link5_radius" value="0.030" />
     <xacro:property name="link6_radius" value="0.025" />
-	<!--   Base Link -->
+<!--   Base Link -->
     <link name="${prefix}base_link" >
       <visual>
@@ -76,17 +66,20 @@
       </xacro:cylinder_inertial>
     </link>
+<xacro:property name="joint1_type" value="revolute"/>
+<xacro:property name="joint1_axe" value="0 0 1"/>
+<xacro:property name="link1_length" value="0.1"/>
 <!--  joint 1	-->
     <joint name="${prefix}joint1" type="${joint1_type}">
       <parent link="${prefix}base_link" />
-      <child link = "${prefix}link1" />
-      <origin xyz="0.0 0.0 ${base_length}" rpy="0.0 0.0 0.0" />
-      <axis xyz="${joint1_axe}" />
+      <child link="${prefix}link1" />
+      <origin xyz="0.0 0.0 ${base_length + link1_length/2}" rpy="0.0 0.0 0.0" />
+      <axis xyz="${joint1_axe}"/>
 	  <xacro:joint_limit joint_type="${joint1_type}" link_length="${link1_length}"/>
       <dynamics damping="0.0" friction="0.0"/>
     </joint>
-<!--  link 1  -->
+    <!--  link 1  -->
     <link name="${prefix}link1">
       <visual>
-		<origin xyz="0 0 ${link1_length/2} " rpy="0 0 0" />
+		<origin xyz="0 0 0 " rpy="0 0 0" />
         <geometry>
 			<cylinder radius="${link1_radius}" length="${link1_length}"/>
@@ -94,23 +87,26 @@
       </visual>
       <collision>
-		 <origin xyz="0 0 ${link1_length/2}" rpy="0 0 0" />
+		 <origin xyz="0 0 ${base_length/2}" rpy="0 0 0" />
         <geometry>
 			<cylinder radius="${link1_radius}" length="${link1_length}"/>
         </geometry>
       </collision>
-      <xacro:cylinder_inertial radius="${link1_length}" length="${link1_length}" mass="${link1_mass}">
+      <xacro:cylinder_inertial radius="${link1_radius}" length="${link1_length}" mass="${link1_mass}">
         <origin xyz="0.0 0.0 ${base_length/2}" rpy="0 0 0" />
       </xacro:cylinder_inertial>
     </link>
+<xacro:property name="joint2_type" value="revolute"/>
+<xacro:property name="joint2_axe" value="0 0 1"/>
+<xacro:property name="link2_length" value="0.4"/>
 <!--  joint 2	-->
     <joint name="${prefix}joint2" type="${joint2_type}">
-      <parent link="${prefix}link1" />
-      <child link = "${prefix}link2" />
-      <origin xyz="0.0 ${link1_radius * 2.0} ${link1_length /2}" rpy="0.0 ${pi / 2.0} 0.0" />
-      <axis xyz="${joint2_axe}" />
+      <parent link="${prefix}link1"/>
+      <child link="${prefix}link2" />
+      <origin xyz="0.0 ${link2_radius + link1_radius} ${link1_length /2}" rpy="${-pi/2} 0 0 "/>
+      <axis xyz="${joint2_axe}"/>
 	  <xacro:joint_limit joint_type="${joint2_type}" link_length="${link2_length}"/>
       <dynamics damping="0.0" friction="0.0"/>
     </joint>
-<!-- link 2	-->
+    <!-- link 2	-->
     <link name="${prefix}link2">
       <visual>
@@ -130,110 +126,122 @@
       </xacro:cylinder_inertial>
     </link>
+<xacro:property name="joint3_type" value="prismatic"/>
+<xacro:property name="joint3_axe" value="0 0 1"/>
+<xacro:property name="link3_length" value="0.7"/>
 <!--  joint 3	-->
     <joint name="${prefix}joint3" type="${joint3_type}">
-      <parent link="${prefix}link2" />
-      <child link = "${prefix}link3" />
-      <origin xyz="0.0 ${link2_radius*2.0} ${link2_length}" rpy="0.0 0.0 0.0" />
-      <axis xyz="${joint3_axe}" />
+      <parent link="${prefix}link2"/>
+      <child link="${prefix}link3" />
+      <origin xyz="0.0 ${link3_radius+link2_radius} ${link2_length}" rpy="0 0 0 "/>
+      <axis xyz="${joint3_axe}"/>
 	  <xacro:joint_limit joint_type="${joint3_type}" link_length="${link3_length}"/>
       <dynamics damping="0.0" friction="0.0"/>
     </joint>
-<!--  link 3 -->
+    <!-- link 3	-->
     <link name="${prefix}link3">
       <visual>
-		<origin xyz="0 0 ${link3_length / 2 }" rpy="0 0 0" />
+		<origin xyz="0 0 ${link3_length / 2}" rpy="0 0 0" />
+        <geometry>
+			<cylinder radius="${link3_radius}" length="${link3_length}"/>
+        </geometry>
+      </visual>
+      <collision>
+	    <origin xyz="0 0 ${link3_length / 2 }" rpy="0 0 0" />
         <geometry>
 		<cylinder radius="${link3_radius}" length="${link3_length}"/>
         </geometry>
-      </visual>
-      <collision>
-		<origin xyz="0 0 ${link3_length / 2 }" rpy="0 0 0" />
-        <geometry>
-			<cylinder radius="${link3_radius}" length="${link3_length}"/>
-        </geometry>
       </collision>
       <xacro:cylinder_inertial radius="${link3_radius}" length="${link3_length}" mass="${link3_mass}">
-        <origin xyz="0 0 ${link3_length / 2 }" rpy="0 0 0" />
-      </xacro:cylinder_inertial>
-    </link>
+        <origin xyz="0.0 0.0 ${link3_length / 2 }" rpy="0 0 0" />
+      </xacro:cylinder_inertial>
+    </link>
+<xacro:property name="joint4_type" value="prismatic"/>
+<xacro:property name="joint4_axe" value="0 0 1"/>
+<xacro:property name="link4_length" value="0.1"/>
 <!--  joint 4	-->
     <joint name="${prefix}joint4" type="${joint4_type}">
-      <parent link="${prefix}link3" />
-      <child link = "${prefix}link4" />
-      <origin xyz="0 -${(link4_radius) * 2 } ${link3_length}" rpy="0.0 0 0.0" />
-      <axis xyz="${joint4_axe} " />
+      <parent link="${prefix}link3"/>
+      <child link="${prefix}link4" />
+      <origin xyz="0 -${link4_radius + link3_radius } ${link3_length}" rpy="${pi/2} 0 0 "/>
+      <axis xyz="${joint4_axe}"/>
 	  <xacro:joint_limit joint_type="${joint4_type}" link_length="${link4_length}"/>
       <dynamics damping="0.0" friction="0.0"/>
     </joint>
-<!-- link 4 -->
+    <!-- link 4	-->
     <link name="${prefix}link4">
       <visual>
-		<origin xyz="0 0 ${link4_length/2}" rpy="0 0 0" />
-        <geometry>
-			   <cylinder radius="${link4_radius}" length="${link4_length}"/>
-        </geometry>
-      </visual>
-      <collision>
-		<origin xyz="0 0 ${link4_length/2}" rpy="0 0 0" />
-        <geometry>
-			   <cylinder radius="${link4_radius}" length="${link4_length}"/>
+		<origin xyz="0 0 ${link4_length / 2}" rpy="0 0 0" />
+        <geometry>
+			<cylinder radius="${link4_radius}" length="${link4_length}"/>
+        </geometry>
+      </visual>
+      <collision>
+	    <origin xyz="0 0 ${link4_length / 2 }" rpy="0 0 0" />
+        <geometry>
+		<cylinder radius="${link4_radius}" length="${link4_length}"/>
         </geometry>
       </collision>
       <xacro:cylinder_inertial radius="${link4_radius}" length="${link4_length}" mass="${link4_mass}">
-        <origin xyz="0 0 ${link4_length/2}" rpy="0 0 0" />
-      </xacro:cylinder_inertial>
-    </link>
+        <origin xyz="0.0 0.0 ${link4_length / 2 }" rpy="0 0 0" />
+      </xacro:cylinder_inertial>
+    </link>
+<xacro:property name="joint5_type" value="revolute"/>
+<xacro:property name="joint5_axe" value="0 0 1"/>
+<xacro:property name="link5_length" value="0.1"/>
 <!--  joint 5	-->
     <joint name="${prefix}joint5" type="${joint5_type}">
-      <parent link="${prefix}link4" />
-      <child link = "${prefix}link5" />
-      <origin xyz="0 0 ${link4_length+link5_radius}" rpy=" ${-pi/2} 0 0" />
-      <axis xyz="${joint5_axe}" />
+      <parent link="${prefix}link4"/>
+      <child link="${prefix}link5" />
+      <origin xyz="0 0 ${link4_length+link5_radius}" rpy="0 0 ${-pi/2} "/>
+      <axis xyz="${joint5_axe}"/>
 	  <xacro:joint_limit joint_type="${joint5_type}" link_length="${link5_length}"/>
       <dynamics damping="0.0" friction="0.0"/>
     </joint>
-<!-- link 5 -->
+    <!-- link 5	-->
     <link name="${prefix}link5">
       <visual>
-        <origin xyz=" 0 0 ${link5_length/2} " rpy="0 0 0" />
+		<origin xyz="0 0 ${link5_length / 2}" rpy="0 0 0" />
+        <geometry>
+			<cylinder radius="${link5_radius}" length="${link5_length}"/>
+        </geometry>
+      </visual>
+      <collision>
+	    <origin xyz="0 0 ${link5_length / 2 }" rpy="0 0 0" />
         <geometry>
 		<cylinder radius="${link5_radius}" length="${link5_length}"/>
         </geometry>
-      </visual>
-      <collision>
-        <origin xyz="0 0 ${link5_length/2} " rpy="0 0 0" />
-        <geometry>
-		<cylinder radius="${link5_radius}" length="${link5_length}"/>
-        </geometry>
       </collision>
       <xacro:cylinder_inertial radius="${link5_radius}" length="${link5_length}" mass="${link5_mass}">
-        <origin xyz="0 0 ${link5_length/2}" rpy="0 0 0" />
-      </xacro:cylinder_inertial>
-    </link>
+        <origin xyz="0.0 0.0 ${link5_length / 2 }" rpy="0 0 0" />
+      </xacro:cylinder_inertial>
+    </link>
+<xacro:property name="joint6_type" value="revolute"/>
+<xacro:property name="joint6_axe" value="0 0 1"/>
+<xacro:property name="link6_length" value="0.1"/>
 <!--  joint 6	-->
     <joint name="${prefix}joint6" type="${joint6_type}">
-      <parent link="${prefix}link5" />
-      <child link = "${prefix}link6" />
-      <origin xyz="0 0 ${link5_length } " rpy="0 0 0" />
-      <axis xyz="${joint6_axe}" />
+      <parent link="${prefix}link5"/>
+      <child link="${prefix}link6" />
+      <origin xyz="0 0 ${link5_length }" rpy="0 0 ${-pi/2} "/>
+      <axis xyz="${joint6_axe}"/>
 	  <xacro:joint_limit joint_type="${joint6_type}" link_length="${link6_length}"/>
       <dynamics damping="0.0" friction="0.0"/>
     </joint>
-<!-- link 6 -->
+    <!-- link 6	-->
     <link name="${prefix}link6">
       <visual>
-        <origin xyz="0 0 ${link6_length/2}" rpy="0 0 0" />
+		<origin xyz="0 0 ${link6_length / 2}" rpy="0 0 0" />
+        <geometry>
+			<cylinder radius="${link6_radius}" length="${link6_length}"/>
+        </geometry>
+      </visual>
+      <collision>
+	    <origin xyz="0 0 ${link6_length / 2 }" rpy="0 0 0" />
         <geometry>
 		<cylinder radius="${link6_radius}" length="${link6_length}"/>
         </geometry>
-      </visual>
-      <collision>
-        <origin xyz="0 0 ${link6_length/2}" rpy="0 0 0" />
-        <geometry>
-		<cylinder radius="${link6_radius}" length="${link6_length}"/>
-        </geometry>
       </collision>
       <xacro:cylinder_inertial radius="${link6_radius}" length="${link6_length}" mass="${link6_mass}">
-        <origin xyz="0 0 ${link6_length/2}" rpy="0 0 0" />
+        <origin xyz="0.0 0.0 ${link6_length / 2 }" rpy="0 0 0" />
       </xacro:cylinder_inertial>
     </link>
@@ -251,13 +259,8 @@
         <origin rpy="0 0 0" xyz="0 0 0.005"/>
       </collision>
-      <visual>
-        <geometry>
-          <box size="0.01 0.01 0.01"/>
-        </geometry>
-        <origin rpy="0 0 0" xyz="0.0 0 0.005"/>
-      </visual>
     </link>
     <xacro:arm_transmission prefix="${prefix}" />
     <xacro:arm_gazebo prefix="${prefix}" />
   </xacro:macro>
+  <xacro:arm_robot prefix=""/>
 </robot>
