Commit message: add 7th dof

File: Manipulator/man_gazebo/urdf/6dof/manipulator6.urdf.xacro (robot description, xacro)
@@ -4,5 +4,5 @@
   <!-- common stuff -->
   <xacro:include filename="$(find man_gazebo)/urdf/common.gazebo.xacro" />
-  <xacro:include filename="$(find man_gazebo)/urdf/manip.urdf.xacro" />
+  <xacro:include filename="$(find man_gazebo)/urdf/manip6.urdf.xacro" />
   <xacro:arm_robot prefix=""/>
 <link name="world" />
@@ -10,5 +10,5 @@
     <parent link="world" />
     <child link = "base_link" />
-    <origin xyz="0 -0.5 0" rpy="0.0 0.0 0.0" />
+    <origin xyz="0 0 0" rpy="0.0 0.0 0.0" />
   </joint>
 </robot>

File: Manipulator/man_gazebo/urdf/6dof/transmission_6dof_6.xacro (robot description, xacro)
@@ -2,14 +2,5 @@
 <robot xmlns:xacro="http://wiki.ros.org/xacro">
   <xacro:macro name="arm_transmission" params="prefix">
- <!-- --> <transmission name="${prefix}joint0_trans">
-      <type>transmission_interface/SimpleTransmission</type>
-      <joint name="${prefix}joint0">
-        <hardwareInterface>hardware_interface/PositionJointInterface</hardwareInterface>
-      </joint>
-      <actuator name="${prefix}joint0_motor">
-        <mechanicalReduction>1</mechanicalReduction>
-      </actuator>
-    </transmission>
- <transmission name="${prefix}joint1_trans">
+    <transmission name="${prefix}joint1_trans">
       <type>transmission_interface/SimpleTransmission</type>
       <joint name="${prefix}joint1">

File: Manipulator/man_gazebo/urdf/gazebo_6.xacro (robot description, xacro)
@@ -20,8 +20,4 @@
 </material>
   <xacro:macro name="arm_gazebo" params="prefix">
-    <gazebo reference="${prefix}link0">
-      <selfCollide>true</selfCollide>
-	  <material>Gazebo/Red</material>
-    </gazebo>
     <gazebo reference="${prefix}link1">
       <selfCollide>true</selfCollide>

File: Manipulator/man_gazebo/urdf/manip.urdf.xacro (robot description, xacro)
@@ -24,4 +24,5 @@
 </xacro:macro>
   <xacro:macro name="arm_robot" params="prefix ">
+	<xacro:property name="joint0_type" value="prismatic" />
     <xacro:property name="joint1_type" value="revolute" />
 	<xacro:property name="joint2_type" value="revolute" />
@@ -30,4 +31,5 @@
 	<xacro:property name="joint5_type" value="revolute" />
 	<xacro:property name="joint6_type" value="revolute" />
+	<xacro:property name="joint0_axe" value="0 0 1" />
 	<xacro:property name="joint1_axe" value="0 0 1" />
 	<xacro:property name="joint2_axe" value="0 1 0" />
@@ -36,6 +38,7 @@
 	<xacro:property name="joint5_axe" value="0 1 0" />
 	<xacro:property name="joint6_axe" value="0 0 1" />
-    <xacro:property name="base_length" value="6.25" />
-	<xacro:property name="link1_length" value="0.15" />
+	<xacro:property name="link0_length" value="0.25" />
+    <xacro:property name="base_length"  value="3.25" />
+	<xacro:property name="link1_length" value="0.25" />
 	<xacro:property name="link2_length" value="0.5" />
 	<xacro:property name="link3_length" value="0.4" />
@@ -44,5 +47,6 @@
 	<xacro:property name="link6_length" value="0.02" />
     <!-- Inertia parameters -->
-    <xacro:property name="base_mass" value="4.0" />
+	<xacro:property name="link0_mass" value="40.7" />
+    <xacro:property name="base_mass" value="1.0" />
     <xacro:property name="link1_mass" value="3.7" />
     <xacro:property name="link2_mass" value="8.393" />
@@ -51,4 +55,5 @@
     <xacro:property name="link5_mass" value="1.219" />
     <xacro:property name="link6_mass" value="0.1879" />
+	<xacro:property name="link0_radius" value="0.060" />
 	<xacro:property name="base_radius" value="0.060" />
     <xacro:property name="link1_radius" value="0.060" />
@@ -76,9 +81,36 @@
       </xacro:cylinder_inertial>
     </link>
+<!--  joint 0	-->
+    <joint name="${prefix}joint0" type="${joint0_type}">
+      <parent link="${prefix}base_link" />
+      <child link = "${prefix}link0" />
+      <origin xyz="0.0 0 ${base_length + link0_radius+0.01}" rpy="${-pi/2} 0.0 0" />
+      <axis xyz="${joint0_axe}" />
+	  <xacro:joint_limit joint_type="${joint0_type}" link_length="${link0_length}"/>
+      <dynamics damping="0.0" friction="0.0"/>
+    </joint>
+<!--  link 0 -->
+    <link name="${prefix}link0">
+      <visual>
+		<origin xyz="0 0 ${link0_radius} " rpy="0 0 0" />
+        <geometry>
+			<cylinder radius="${link0_radius}" length="${link0_length}"/>
+        </geometry>
+      </visual>
+      <collision>
+		 <origin xyz="0 0 ${link0_radius}" rpy="0 0 0" />
+        <geometry>
+			<cylinder radius="${link0_radius}" length="${link0_length}"  mass="${link0_mass}"/>
+        </geometry>
+      </collision>
+      <xacro:cylinder_inertial radius="${link0_radius}" length="${link0_length}" mass="${link0_mass}">
+        <origin xyz="0.0 0.0 ${link0_radius}" rpy="0 0 0" />
+      </xacro:cylinder_inertial>
+    </link>
 <!--  joint 1	-->
     <joint name="${prefix}joint1" type="${joint1_type}">
-      <parent link="${prefix}base_link" />
+      <parent link="${prefix}link0" />
       <child link = "${prefix}link1" />
-      <origin xyz="0.0 0.0 ${base_length}" rpy="0.0 0.0 ${-pi/2}" />
+      <origin xyz="0.0 0.0 ${link0_length}" rpy="0.0 0 -${pi/2}" />
       <axis xyz="${joint1_axe}" />
 	  <xacro:joint_limit joint_type="${joint1_type}" link_length="${link1_length}"/>
@@ -107,5 +139,5 @@
       <parent link="${prefix}link1" />
       <child link = "${prefix}link2" />
-      <origin xyz="0.0 ${link1_radius * 2.0} ${link1_length /2}" rpy="0.0 ${pi / 2.0} 0.0" />
+      <origin xyz="0.0 ${link1_radius * 2.0} ${link1_length }" rpy="0.0 ${pi/2.0} 0.0" />
       <axis xyz="${joint2_axe}" />
 	  <xacro:joint_limit joint_type="${joint2_type}" link_length="${link2_length}"/>
@@ -161,5 +193,5 @@
       <parent link="${prefix}link3" />
       <child link = "${prefix}link4" />
-      <origin xyz="0 -${(link4_radius) * 2 } ${link3_length}" rpy="0.0 0 0.0" />
+      <origin xyz="0 -${link4_radius + link3_radius } ${link3_length}" rpy="0.0 0 0.0" />
       <axis xyz="${joint4_axe} " />
 	  <xacro:joint_limit joint_type="${joint4_type}" link_length="${link4_length}"/>

File: Manipulator/man_gazebo/urdf/manip6.urdf.xacro (robot description, xacro)
@@ -1,14 +1,6 @@
 <?xml version="1.0"?>
-<robot xmlns:xacro="http://wiki.ros.org/xacro" name="arm" >
-<!-- common stuff -->
-<xacro:include filename="$(find man_gazebo)/urdf/common.gazebo.xacro" />
-<link name="world" />
-  <joint name="world_joint" type="fixed">
-    <parent link="world" />
-    <child link = "base_link" />
-    <origin xyz="0 0 0" rpy="0.0 0.0 0.0" />
-  </joint>
-  <xacro:include filename="$(find man_gazebo)/urdf/transmission.xacro" />
-  <xacro:include filename="$(find man_gazebo)/urdf/gazebo.xacro" />
+<robot xmlns:xacro="http://wiki.ros.org/xacro">
+  <xacro:include filename="$(find man_gazebo)/urdf/6dof/transmission_6dof_6.xacro" />
+  <xacro:include filename="$(find man_gazebo)/urdf/gazebo_6.xacro" />
   <xacro:macro name="cylinder_inertial" params="radius length mass *origin">
     <inertial>
@@ -32,5 +24,23 @@
 </xacro:macro>
   <xacro:macro name="arm_robot" params="prefix ">
-    <xacro:property name="base_length" value="0.25" />
+    <xacro:property name="joint1_type" value="revolute" />
+	<xacro:property name="joint2_type" value="revolute" />
+	<xacro:property name="joint3_type" value="revolute" />
+	<xacro:property name="joint4_type" value="revolute" />
+	<xacro:property name="joint5_type" value="revolute" />
+	<xacro:property name="joint6_type" value="revolute" />
+	<xacro:property name="joint1_axe" value="0 0 1" />
+	<xacro:property name="joint2_axe" value="0 1 0" />
+	<xacro:property name="joint3_axe" value="0 1 0" />
+	<xacro:property name="joint4_axe" value="0 1 0" />
+	<xacro:property name="joint5_axe" value="0 1 0" />
+	<xacro:property name="joint6_axe" value="0 0 1" />
+    <xacro:property name="base_length" value="3.25" />
+	<xacro:property name="link1_length" value="0.15" />
+	<xacro:property name="link2_length" value="0.5" />
+	<xacro:property name="link3_length" value="0.4" />
+	<xacro:property name="link4_length" value="0.07" />
+	<xacro:property name="link5_length" value="0.1" />
+	<xacro:property name="link6_length" value="0.02" />
     <!-- Inertia parameters -->
     <xacro:property name="base_mass" value="4.0" />
@@ -48,5 +58,5 @@
     <xacro:property name="link5_radius" value="0.030" />
     <xacro:property name="link6_radius" value="0.025" />
-<!--   Base Link -->
+	<!--   Base Link -->
     <link name="${prefix}base_link" >
       <visual>
@@ -66,20 +76,17 @@
       </xacro:cylinder_inertial>
     </link>
-<xacro:property name="joint1_type" value="revolute"/>
-<xacro:property name="joint1_axe" value="0 0 1"/>
-<xacro:property name="link1_length" value="0.1"/>
 <!--  joint 1	-->
     <joint name="${prefix}joint1" type="${joint1_type}">
       <parent link="${prefix}base_link" />
-      <child link="${prefix}link1" />
-      <origin xyz="0.0 0.0 ${base_length + link1_length/2}" rpy="0.0 0.0 0.0" />
-      <axis xyz="${joint1_axe}"/>
+      <child link = "${prefix}link1" />
+      <origin xyz="0.0 0.0 ${base_length}" rpy="0.0 0.0 ${-pi/2}" />
+      <axis xyz="${joint1_axe}" />
 	  <xacro:joint_limit joint_type="${joint1_type}" link_length="${link1_length}"/>
       <dynamics damping="0.0" friction="0.0"/>
     </joint>
-    <!--  link 1  -->
+<!--  link 1  -->
     <link name="${prefix}link1">
       <visual>
-		<origin xyz="0 0 0 " rpy="0 0 0" />
+		<origin xyz="0 0 ${link1_length/2} " rpy="0 0 0" />
         <geometry>
 			<cylinder radius="${link1_radius}" length="${link1_length}"/>
@@ -87,26 +94,23 @@
       </visual>
       <collision>
-		 <origin xyz="0 0 ${base_length/2}" rpy="0 0 0" />
-        <geometry>
-			<cylinder radius="${link1_radius}" length="${link1_length}"/>
+		 <origin xyz="0 0 ${link1_length/2}" rpy="0 0 0" />
+        <geometry>
+			<cylinder radius="${link1_radius}" length="${link1_length}"  mass="${link1_mass}"/>
         </geometry>
       </collision>
       <xacro:cylinder_inertial radius="${link1_radius}" length="${link1_length}" mass="${link1_mass}">
-        <origin xyz="0.0 0.0 ${base_length/2}" rpy="0 0 0" />
-      </xacro:cylinder_inertial>
-    </link>
-<xacro:property name="joint2_type" value="revolute"/>
-<xacro:property name="joint2_axe" value="0 0 1"/>
-<xacro:property name="link2_length" value="0.4"/>
+        <origin xyz="0.0 0.0 ${link1_length/2}" rpy="0 0 0" />
+      </xacro:cylinder_inertial>
+    </link>
 <!--  joint 2	-->
     <joint name="${prefix}joint2" type="${joint2_type}">
-      <parent link="${prefix}link1"/>
-      <child link="${prefix}link2" />
-      <origin xyz="0.0 ${link2_radius + link1_radius} ${link1_length /2}" rpy="${-pi/2} 0 0 "/>
-      <axis xyz="${joint2_axe}"/>
+      <parent link="${prefix}link1" />
+      <child link = "${prefix}link2" />
+      <origin xyz="0.0 ${link1_radius * 2.0} ${link1_length /2}" rpy="0.0 ${pi / 2.0} 0.0" />
+      <axis xyz="${joint2_axe}" />
 	  <xacro:joint_limit joint_type="${joint2_type}" link_length="${link2_length}"/>
       <dynamics damping="0.0" friction="0.0"/>
     </joint>
-    <!-- link 2	-->
+<!-- link 2	-->
     <link name="${prefix}link2">
       <visual>
@@ -126,122 +130,110 @@
       </xacro:cylinder_inertial>
     </link>
-<xacro:property name="joint3_type" value="prismatic"/>
-<xacro:property name="joint3_axe" value="0 0 1"/>
-<xacro:property name="link3_length" value="0.7"/>
 <!--  joint 3	-->
     <joint name="${prefix}joint3" type="${joint3_type}">
-      <parent link="${prefix}link2"/>
-      <child link="${prefix}link3" />
-      <origin xyz="0.0 ${link3_radius+link2_radius} ${link2_length}" rpy="0 0 0 "/>
-      <axis xyz="${joint3_axe}"/>
+      <parent link="${prefix}link2" />
+      <child link = "${prefix}link3" />
+      <origin xyz="0.0 ${link2_radius*2.0} ${link2_length}" rpy="0.0 0.0 0.0" />
+      <axis xyz="${joint3_axe}" />
 	  <xacro:joint_limit joint_type="${joint3_type}" link_length="${link3_length}"/>
       <dynamics damping="0.0" friction="0.0"/>
     </joint>
-    <!-- link 3	-->
+<!--  link 3 -->
     <link name="${prefix}link3">
       <visual>
-		<origin xyz="0 0 ${link3_length / 2}" rpy="0 0 0" />
+		<origin xyz="0 0 ${link3_length / 2 }" rpy="0 0 0" />
+        <geometry>
+		<cylinder radius="${link3_radius}" length="${link3_length}"/>
+        </geometry>
+      </visual>
+      <collision>
+		<origin xyz="0 0 ${link3_length / 2 }" rpy="0 0 0" />
         <geometry>
 			<cylinder radius="${link3_radius}" length="${link3_length}"/>
         </geometry>
-      </visual>
-      <collision>
-	    <origin xyz="0 0 ${link3_length / 2 }" rpy="0 0 0" />
-        <geometry>
-		<cylinder radius="${link3_radius}" length="${link3_length}"/>
-        </geometry>
       </collision>
       <xacro:cylinder_inertial radius="${link3_radius}" length="${link3_length}" mass="${link3_mass}">
-        <origin xyz="0.0 0.0 ${link3_length / 2 }" rpy="0 0 0" />
-      </xacro:cylinder_inertial>
-    </link>
-<xacro:property name="joint4_type" value="prismatic"/>
-<xacro:property name="joint4_axe" value="0 0 1"/>
-<xacro:property name="link4_length" value="0.1"/>
+        <origin xyz="0 0 ${link3_length / 2 }" rpy="0 0 0" />
+      </xacro:cylinder_inertial>
+    </link>
 <!--  joint 4	-->
     <joint name="${prefix}joint4" type="${joint4_type}">
-      <parent link="${prefix}link3"/>
-      <child link="${prefix}link4" />
-      <origin xyz="0 -${link4_radius + link3_radius } ${link3_length}" rpy="${pi/2} 0 0 "/>
-      <axis xyz="${joint4_axe}"/>
+      <parent link="${prefix}link3" />
+      <child link = "${prefix}link4" />
+      <origin xyz="0 -${(link4_radius) * 2 } ${link3_length}" rpy="0.0 0 0.0" />
+      <axis xyz="${joint4_axe} " />
 	  <xacro:joint_limit joint_type="${joint4_type}" link_length="${link4_length}"/>
       <dynamics damping="0.0" friction="0.0"/>
     </joint>
-    <!-- link 4	-->
+<!-- link 4 -->
     <link name="${prefix}link4">
       <visual>
-		<origin xyz="0 0 ${link4_length / 2}" rpy="0 0 0" />
-        <geometry>
-			<cylinder radius="${link4_radius}" length="${link4_length}"/>
-        </geometry>
-      </visual>
-      <collision>
-	    <origin xyz="0 0 ${link4_length / 2 }" rpy="0 0 0" />
-        <geometry>
-		<cylinder radius="${link4_radius}" length="${link4_length}"/>
+		<origin xyz="0 0 ${link4_length/2}" rpy="0 0 0" />
+        <geometry>
+			   <cylinder radius="${link4_radius}" length="${link4_length}"/>
+        </geometry>
+      </visual>
+      <collision>
+		<origin xyz="0 0 ${link4_length/2}" rpy="0 0 0" />
+        <geometry>
+			   <cylinder radius="${link4_radius}" length="${link4_length}"/>
         </geometry>
       </collision>
       <xacro:cylinder_inertial radius="${link4_radius}" length="${link4_length}" mass="${link4_mass}">
-        <origin xyz="0.0 0.0 ${link4_length / 2 }" rpy="0 0 0" />
-      </xacro:cylinder_inertial>
-    </link>
-<xacro:property name="joint5_type" value="revolute"/>
-<xacro:property name="joint5_axe" value="0 0 1"/>
-<xacro:property name="link5_length" value="0.1"/>
+        <origin xyz="0 0 ${link4_length/2}" rpy="0 0 0" />
+      </xacro:cylinder_inertial>
+    </link>
 <!--  joint 5	-->
     <joint name="${prefix}joint5" type="${joint5_type}">
-      <parent link="${prefix}link4"/>
-      <child link="${prefix}link5" />
-      <origin xyz="0 0 ${link4_length+link5_radius}" rpy="0 0 ${-pi/2} "/>
-      <axis xyz="${joint5_axe}"/>
+      <parent link="${prefix}link4" />
+      <child link = "${prefix}link5" />
+      <origin xyz="0 0 ${link4_length+link5_radius}" rpy=" ${-pi/2} 0 0" />
+      <axis xyz="${joint5_axe}" />
 	  <xacro:joint_limit joint_type="${joint5_type}" link_length="${link5_length}"/>
       <dynamics damping="0.0" friction="0.0"/>
     </joint>
-    <!-- link 5	-->
+<!-- link 5 -->
     <link name="${prefix}link5">
       <visual>
-		<origin xyz="0 0 ${link5_length / 2}" rpy="0 0 0" />
-        <geometry>
-			<cylinder radius="${link5_radius}" length="${link5_length}"/>
-        </geometry>
-      </visual>
-      <collision>
-	    <origin xyz="0 0 ${link5_length / 2 }" rpy="0 0 0" />
+        <origin xyz=" 0 0 ${link5_length/2} " rpy="0 0 0" />
         <geometry>
 		<cylinder radius="${link5_radius}" length="${link5_length}"/>
         </geometry>
+      </visual>
+      <collision>
+        <origin xyz="0 0 ${link5_length/2} " rpy="0 0 0" />
+        <geometry>
+		<cylinder radius="${link5_radius}" length="${link5_length}"/>
+        </geometry>
       </collision>
       <xacro:cylinder_inertial radius="${link5_radius}" length="${link5_length}" mass="${link5_mass}">
-        <origin xyz="0.0 0.0 ${link5_length / 2 }" rpy="0 0 0" />
-      </xacro:cylinder_inertial>
-    </link>
-<xacro:property name="joint6_type" value="revolute"/>
-<xacro:property name="joint6_axe" value="0 0 1"/>
-<xacro:property name="link6_length" value="0.1"/>
+        <origin xyz="0 0 ${link5_length/2}" rpy="0 0 0" />
+      </xacro:cylinder_inertial>
+    </link>
 <!--  joint 6	-->
     <joint name="${prefix}joint6" type="${joint6_type}">
-      <parent link="${prefix}link5"/>
-      <child link="${prefix}link6" />
-      <origin xyz="0 0 ${link5_length }" rpy="0 0 ${-pi/2} "/>
-      <axis xyz="${joint6_axe}"/>
+      <parent link="${prefix}link5" />
+      <child link = "${prefix}link6" />
+      <origin xyz="0 0 ${link5_length } " rpy="0 0 0" />
+      <axis xyz="${joint6_axe}" />
 	  <xacro:joint_limit joint_type="${joint6_type}" link_length="${link6_length}"/>
       <dynamics damping="0.0" friction="0.0"/>
     </joint>
-    <!-- link 6	-->
+<!-- link 6 -->
     <link name="${prefix}link6">
       <visual>
-		<origin xyz="0 0 ${link6_length / 2}" rpy="0 0 0" />
-        <geometry>
-			<cylinder radius="${link6_radius}" length="${link6_length}"/>
-        </geometry>
-      </visual>
-      <collision>
-	    <origin xyz="0 0 ${link6_length / 2 }" rpy="0 0 0" />
+        <origin xyz="0 0 ${link6_length/2}" rpy="0 0 0" />
         <geometry>
 		<cylinder radius="${link6_radius}" length="${link6_length}"/>
         </geometry>
+      </visual>
+      <collision>
+        <origin xyz="0 0 ${link6_length/2}" rpy="0 0 0" />
+        <geometry>
+		<cylinder radius="${link6_radius}" length="${link6_length}"/>
+        </geometry>
       </collision>
       <xacro:cylinder_inertial radius="${link6_radius}" length="${link6_length}" mass="${link6_mass}">
-        <origin xyz="0.0 0.0 ${link6_length / 2 }" rpy="0 0 0" />
+        <origin xyz="0 0 ${link6_length/2}" rpy="0 0 0" />
       </xacro:cylinder_inertial>
     </link>
@@ -259,8 +251,13 @@
         <origin rpy="0 0 0" xyz="0 0 0.005"/>
       </collision>
+      <visual>
+        <geometry>
+          <box size="0.01 0.01 0.01"/>
+        </geometry>
+        <origin rpy="0 0 0" xyz="0.0 0 0.005"/>
+      </visual>
     </link>
     <xacro:arm_transmission prefix="${prefix}" />
     <xacro:arm_gazebo prefix="${prefix}" />
   </xacro:macro>
-  <xacro:arm_robot prefix=""/>
 </robot>
