Commit message: cancel roll in final joint

File: Manipulator/man_gazebo/urdf/6dof/manipulator.urdf.xacro (robot description, xacro)
@@ -10,5 +10,5 @@
     <parent link="world" />
     <child link = "base_link" />
-    <origin xyz="0 -0.5 0" rpy="0.0 0.0 0.0" />
+    <origin xyz="0 -1 0" rpy="0.0 0.0 0.0" />
   </joint>
 </robot>

File: Manipulator/man_gazebo/urdf/6dof/transmission_6dof.xacro (robot description, xacro)
@@ -65,13 +65,4 @@
       </actuator>
     </transmission>
-   <transmission name="${prefix}ee_joint_trans">
-      <type>transmission_interface/SimpleTransmission</type>
-      <joint name="${prefix}ee_joint">
-        <hardwareInterface>hardware_interface/PositionJointInterface</hardwareInterface>
-      </joint>
-      <actuator name="${prefix}ee_joint_motor">
-        <mechanicalReduction>1</mechanicalReduction>
-      </actuator>
-    </transmission>
   </xacro:macro>
 </robot>

File: Manipulator/man_gazebo/urdf/manip.urdf.xacro (robot description, xacro)
@@ -87,5 +87,5 @@
       <origin xyz="0.0 0 ${base_length + link0_radius+0.01}" rpy="${-pi/2} 0.0 0" />
       <axis xyz="${joint0_axe}" />
-	  <xacro:joint_limit joint_type="${joint0_type}" link_length="${link0_length}"/>
+	  <xacro:joint_limit joint_type="${joint0_type}" link_length="${link0_length*6}"/>
       <dynamics damping="0.0" friction="0.0"/>
     </joint>
@@ -270,11 +270,8 @@
       </xacro:cylinder_inertial>
     </link>
-    <joint name="${prefix}ee_joint" type="revolute">
+    <joint name="${prefix}ee_fixed_joint" type="fixed">
       <parent link="${prefix}link6" />
       <child link = "${prefix}ee_link" />
       <origin xyz="0.0  0.0 ${link6_length}" rpy="0.0 0.0 0" />
-      <axis xyz="0 0 1"/>
-      <xacro:joint_limit joint_type="revolute" link_length="0.1"/>
-      <dynamics damping="0.0" friction="0.0"/>
     </joint>
 <!-- ee link -->
@@ -286,8 +283,5 @@
         <origin rpy="0 0 0" xyz="0 0 0.005"/>
       </collision>
-      <xacro:cylinder_inertial radius="0.01" length="0.01" mass="0.01">
-        <origin xyz="0.0 0.0 0.005" rpy="0 0 0" />
-      </xacro:cylinder_inertial>
-    </link>
+	</link>
     <xacro:arm_transmission prefix="${prefix}" />
     <xacro:arm_gazebo prefix="${prefix}" />

Commit message: fix 6dof default manipulator

File: Manipulator/man_gazebo/urdf/6dof/manipulator.urdf.xacro (robot description, xacro)
@@ -1,9 +1,8 @@
 <?xml version="1.0"?>
-<robot xmlns:xacro="http://wiki.ros.org/xacro"
-       name="arm" >
+<robot xmlns:xacro="http://wiki.ros.org/xacro"  name="arm" >
   <!-- common stuff -->
   <xacro:include filename="$(find man_gazebo)/urdf/common.gazebo.xacro" />
-  <xacro:include filename="$(find man_gazebo)/urdf/manip.urdf.xacro" />
-  <xacro:arm_robot prefix=""/>
+ <xacro:include filename="$(find man_gazebo)/urdf/6dof/transmission_6dof.xacro" />
+  <xacro:include filename="$(find man_gazebo)/urdf/gazebo.xacro" />
 <link name="world" />
   <joint name="world_joint" type="fixed">
@@ -12,3 +11,309 @@
     <origin xyz="0 -1 0" rpy="0.0 0.0 0.0" />
   </joint>
+  <xacro:macro name="cylinder_inertial" params="radius length mass *origin">
+    <inertial>
+      <mass value="${mass}" />
+      <xacro:insert_block name="origin" />
+      <inertia ixx="${0.0833333 * mass * (3 * radius * radius + length * length)}" ixy="0.0" ixz="0.0"
+        iyy="${0.0833333 * mass * (3 * radius * radius + length * length)}" iyz="0.0"
+        izz="${0.5 * mass * radius * radius}" />
+    </inertial>
+  </xacro:macro>
+<xacro:macro name="joint_limit" params="joint_type link_length ">
+	<xacro:if value="${joint_type == 'revolute'}"  >
+		<xacro:property name="joint_upper_limit" value="${pi}" />
+		<xacro:property name="joint_lower_limit" value="${-pi}" />
+	</xacro:if>
+	<xacro:unless value="${joint_type == 'revolute'}"  >
+		<xacro:property name="joint_upper_limit" value="${2*link_length}" />
+		<xacro:property name="joint_lower_limit" value="${0}" />
+	</xacro:unless>
+	<limit lower="${joint_lower_limit}" upper="${joint_upper_limit}" effort="150.0" velocity="3.15"/>
+</xacro:macro>
+<xacro:macro name="arm_robot" params="prefix ">
+	<xacro:property name="joint0_type" value="prismatic" />
+    <xacro:property name="joint1_type" value="revolute" />
+	<xacro:property name="joint2_type" value="revolute" />
+	<xacro:property name="joint3_type" value="revolute" />
+	<xacro:property name="joint4_type" value="revolute" />
+	<xacro:property name="joint5_type" value="revolute" />
+	<xacro:property name="joint6_type" value="revolute" />
+	<xacro:property name="joint0_axe" value="0 0 1" />
+	<xacro:property name="joint1_axe" value="0 0 1" />
+	<xacro:property name="joint2_axe" value="0 1 0" />
+	<xacro:property name="joint3_axe" value="0 1 0" />
+	<xacro:property name="joint4_axe" value="0 1 0" />
+	<xacro:property name="joint5_axe" value="0 1 0" />
+	<xacro:property name="joint6_axe" value="0 0 1" />
+	<xacro:property name="link0_length" value="0.25" />
+    <xacro:property name="base_length"  value="3.25" />
+	<xacro:property name="link1_length" value="0.25" />
+	<xacro:property name="link2_length" value="0.5" />
+	<xacro:property name="link3_length" value="0.4" />
+	<xacro:property name="link4_length" value="0.07" />
+	<xacro:property name="link5_length" value="0.1" />
+	<xacro:property name="link6_length" value="0.02" />
+    <!-- Inertia parameters -->
+	<xacro:property name="link0_mass" value="40.7" />
+    <xacro:property name="base_mass" value="1.0" />
+    <xacro:property name="link1_mass" value="3.7" />
+    <xacro:property name="link2_mass" value="8.393" />
+    <xacro:property name="link3_mass" value="2.275" />
+    <xacro:property name="link4_mass" value="1.219" />
+    <xacro:property name="link5_mass" value="1.219" />
+    <xacro:property name="link6_mass" value="0.1879" />
+	<xacro:property name="link0_radius" value="0.060" />
+	<xacro:property name="base_radius" value="0.060" />
+    <xacro:property name="link1_radius" value="0.060" />
+    <xacro:property name="link2_radius" value="0.060" />
+    <xacro:property name="link3_radius" value="0.060" />
+    <xacro:property name="link4_radius" value="0.040" />
+    <xacro:property name="link5_radius" value="0.030" />
+    <xacro:property name="link6_radius" value="0.025" />
+	<!--   Base Link -->
+    <link name="${prefix}base_link" >
+      <visual>
+		<origin xyz="0 0 ${base_length/2}" rpy="0 0 0" />
+        <geometry>
+ 			<cylinder radius="${base_radius}" length="${base_length}"/>
+        </geometry>
+      </visual>
+      <collision>
+			<origin xyz="0 0 ${base_length/2}" rpy="0 0 0" />
+        <geometry>
+			<cylinder radius="${base_radius}" length="${base_length}"/>
+        </geometry>
+      </collision>
+      <xacro:cylinder_inertial radius="${base_radius}" length="${base_length}" mass="${base_mass}">
+        <origin xyz="0.0 0.0 ${base_length/2}" rpy="0 0 0" />
+      </xacro:cylinder_inertial>
+    </link>
+<!--  joint 0	-->
+    <joint name="${prefix}joint0" type="${joint0_type}">
+      <parent link="${prefix}base_link" />
+      <child link = "${prefix}link0" />
+      <origin xyz="0.0 0 ${base_length + link0_radius+0.01}" rpy="${-pi/2} 0.0 0" />
+      <axis xyz="${joint0_axe}" />
+	  <xacro:joint_limit joint_type="${joint0_type}" link_length="${link0_length*6}"/>
+      <dynamics damping="0.0" friction="0.0"/>
+    </joint>
+<!--  link 0 -->
+    <link name="${prefix}link0">
+      <visual>
+		<origin xyz="0 0 ${link0_radius} " rpy="0 0 0" />
+        <geometry>
+			<cylinder radius="${link0_radius}" length="${link0_length}"/>
+        </geometry>
+      </visual>
+      <collision>
+		 <origin xyz="0 0 ${link0_radius}" rpy="0 0 0" />
+        <geometry>
+			<cylinder radius="${link0_radius}" length="${link0_length}"  mass="${link0_mass}"/>
+        </geometry>
+      </collision>
+      <xacro:cylinder_inertial radius="${link0_radius}" length="${link0_length}" mass="${link0_mass}">
+        <origin xyz="0.0 0.0 ${link0_radius}" rpy="0 0 0" />
+      </xacro:cylinder_inertial>
+    </link>
+<!--  joint 1	-->
+    <joint name="${prefix}joint1" type="${joint1_type}">
+      <parent link="${prefix}link0" />
+      <child link = "${prefix}link1" />
+      <origin xyz="0.0 0.0 ${link0_length}" rpy="${pi/2} 0 0" />
+      <axis xyz="${joint1_axe}" />
+	  <xacro:joint_limit joint_type="${joint1_type}" link_length="${link1_length}"/>
+      <dynamics damping="0.0" friction="0.0"/>
+    </joint>
+<!--  link 1  -->
+    <link name="${prefix}link1">
+      <visual>
+		<origin xyz="0 0 ${link1_length/2} " rpy="0 0 0" />
+        <geometry>
+			<cylinder radius="${link1_radius}" length="${link1_length}"/>
+        </geometry>
+      </visual>
+      <collision>
+		 <origin xyz="0 0 ${link1_length/2}" rpy="0 0 0" />
+        <geometry>
+			<cylinder radius="${link1_radius}" length="${link1_length}"  mass="${link1_mass}"/>
+        </geometry>
+      </collision>
+      <xacro:cylinder_inertial radius="${link1_radius}" length="${link1_length}" mass="${link1_mass}">
+        <origin xyz="0.0 0.0 ${link1_length/2}" rpy="0 0 0" />
+      </xacro:cylinder_inertial>
+    </link>
+<!--  joint 2	-->
+    <joint name="${prefix}joint2" type="${joint2_type}">
+      <parent link="${prefix}link1" />
+      <child link = "${prefix}link2" />
+      <origin xyz="0.0 ${link1_radius * 2.0} ${link1_length }" rpy="0.0 ${pi/2.0} 0.0" />
+      <axis xyz="${joint2_axe}" />
+	  <xacro:joint_limit joint_type="${joint2_type}" link_length="${link2_length}"/>
+      <dynamics damping="0.0" friction="0.0"/>
+    </joint>
+<!-- link 2	-->
+    <link name="${prefix}link2">
+      <visual>
+		<origin xyz="0 0 ${link2_length / 2}" rpy="0 0 0" />
+        <geometry>
+			<cylinder radius="${link2_radius}" length="${link2_length}"/>
+        </geometry>
+      </visual>
+      <collision>
+	    <origin xyz="0 0 ${link2_length / 2 }" rpy="0 0 0" />
+        <geometry>
+		<cylinder radius="${link2_radius}" length="${link2_length}"/>
+        </geometry>
+      </collision>
+      <xacro:cylinder_inertial radius="${link2_radius}" length="${link2_length}" mass="${link2_mass}">
+        <origin xyz="0.0 0.0 ${link2_length / 2 }" rpy="0 0 0" />
+      </xacro:cylinder_inertial>
+    </link>
+<!--  joint 3	-->
+    <joint name="${prefix}joint3" type="${joint3_type}">
+      <parent link="${prefix}link2" />
+      <child link = "${prefix}link3" />
+      <origin xyz="0.0 ${link2_radius*2.0} ${link2_length}" rpy="0.0 0.0 0.0" />
+      <axis xyz="${joint3_axe}" />
+	  <xacro:joint_limit joint_type="${joint3_type}" link_length="${link3_length}"/>
+      <dynamics damping="0.0" friction="0.0"/>
+    </joint>
+<!--  link 3 -->
+    <link name="${prefix}link3">
+      <visual>
+		<origin xyz="0 0 ${link3_length / 2 }" rpy="0 0 0" />
+        <geometry>
+		<cylinder radius="${link3_radius}" length="${link3_length}"/>
+        </geometry>
+      </visual>
+      <collision>
+		<origin xyz="0 0 ${link3_length / 2 }" rpy="0 0 0" />
+        <geometry>
+			<cylinder radius="${link3_radius}" length="${link3_length}"/>
+        </geometry>
+      </collision>
+      <xacro:cylinder_inertial radius="${link3_radius}" length="${link3_length}" mass="${link3_mass}">
+        <origin xyz="0 0 ${link3_length / 2 }" rpy="0 0 0" />
+      </xacro:cylinder_inertial>
+    </link>
+<!--  joint 4	-->
+    <joint name="${prefix}joint4" type="${joint4_type}">
+      <parent link="${prefix}link3" />
+      <child link = "${prefix}link4" />
+      <origin xyz="0 -${link4_radius + link3_radius } ${link3_length}" rpy="0.0 0 0.0" />
+      <axis xyz="${joint4_axe} " />
+	  <xacro:joint_limit joint_type="${joint4_type}" link_length="${link4_length}"/>
+      <dynamics damping="0.0" friction="0.0"/>
+    </joint>
+<!-- link 4 -->
+    <link name="${prefix}link4">
+      <visual>
+		<origin xyz="0 0 ${link4_length/2}" rpy="0 0 0" />
+        <geometry>
+			   <cylinder radius="${link4_radius}" length="${link4_length}"/>
+        </geometry>
+      </visual>
+      <collision>
+		<origin xyz="0 0 ${link4_length/2}" rpy="0 0 0" />
+        <geometry>
+			   <cylinder radius="${link4_radius}" length="${link4_length}"/>
+        </geometry>
+      </collision>
+      <xacro:cylinder_inertial radius="${link4_radius}" length="${link4_length}" mass="${link4_mass}">
+        <origin xyz="0 0 ${link4_length/2}" rpy="0 0 0" />
+      </xacro:cylinder_inertial>
+    </link>
+<!--  joint 5	-->
+    <joint name="${prefix}joint5" type="${joint5_type}">
+      <parent link="${prefix}link4" />
+      <child link = "${prefix}link5" />
+      <origin xyz="0 0 ${link4_length+link5_radius}" rpy=" ${-pi/2} 0 0" />
+      <axis xyz="${joint5_axe}" />
+	  <xacro:joint_limit joint_type="${joint5_type}" link_length="${link5_length}"/>
+      <dynamics damping="0.0" friction="0.0"/>
+    </joint>
+<!-- link 5 -->
+    <link name="${prefix}link5">
+      <visual>
+        <origin xyz=" 0 0 ${link5_length/2} " rpy="0 0 0" />
+        <geometry>
+		<cylinder radius="${link5_radius}" length="${link5_length}"/>
+        </geometry>
+      </visual>
+      <collision>
+        <origin xyz="0 0 ${link5_length/2} " rpy="0 0 0" />
+        <geometry>
+		<cylinder radius="${link5_radius}" length="${link5_length}"/>
+        </geometry>
+      </collision>
+      <xacro:cylinder_inertial radius="${link5_radius}" length="${link5_length}" mass="${link5_mass}">
+        <origin xyz="0 0 ${link5_length/2}" rpy="0 0 0" />
+      </xacro:cylinder_inertial>
+    </link>
+<!--  joint 6	-->
+    <joint name="${prefix}joint6" type="${joint6_type}">
+      <parent link="${prefix}link5" />
+      <child link = "${prefix}link6" />
+      <origin xyz="0 0 ${link5_length } " rpy="0 0 0" />
+      <axis xyz="${joint6_axe}" />
+	  <xacro:joint_limit joint_type="${joint6_type}" link_length="${link6_length}"/>
+      <dynamics damping="0.0" friction="0.0"/>
+    </joint>
+<!-- link 6 -->
+    <link name="${prefix}link6">
+      <visual>
+        <origin xyz="0 0 ${link6_length/2}" rpy="0 0 0" />
+        <geometry>
+		<cylinder radius="${link6_radius}" length="${link6_length}"/>
+        </geometry>
+      </visual>
+      <collision>
+        <origin xyz="0 0 ${link6_length/2}" rpy="0 0 0" />
+        <geometry>
+		<cylinder radius="${link6_radius}" length="${link6_length}"/>
+        </geometry>
+      </collision>
+      <xacro:cylinder_inertial radius="${link6_radius}" length="${link6_length}" mass="${link6_mass}">
+        <origin xyz="0 0 ${link6_length/2}" rpy="0 0 0" />
+      </xacro:cylinder_inertial>
+    </link>
+         <!-- fake joint - the rotation about z axe of the camera is not important -->
+        <joint name="fake_joint" type="revolute">
+      <parent link="${prefix}link6" />
+      <child link = "camera_link" />
+      <origin xyz="0.0  0.0 ${link6_length}" rpy="0.0 0.0 0" />
+      <axis xyz="0 0 1"/>
+      <xacro:joint_limit joint_type="revolute" link_length="0.1"/>
+      <dynamics damping="0.0" friction="0.0"/>
+        </joint>
+    <!-- camera link -->
+        <link name="camera_link">
+          <collision>
+            <geometry>
+              <box size="0.01 0.01 0.01"/>
+            </geometry>
+            <origin rpy="0 0 0" xyz="0 0 0.005"/>
+          </collision>
+          <xacro:cylinder_inertial radius="0.01" length="0.01" mass="0.01">
+            <origin xyz="0.0 0.0 0.005" rpy="0 0 0" />
+          </xacro:cylinder_inertial>
+        </link>
+    <joint name="${prefix}ee_fixed_joint" type="fixed">
+      <parent link="${prefix}camera_link" />
+      <child link = "${prefix}ee_link" />
+      <origin xyz="0.0  0.0 0.01" rpy="0.0 0.0 0" />
+    </joint>
+<!-- ee link -->
+    <link name="${prefix}ee_link">
+      <collision>
+        <geometry>
+          <box size="0.01 0.01 0.01"/>
+        </geometry>
+        <origin rpy="0 0 0" xyz="0 0 0.005"/>
+      </collision>
+	</link>
+    <xacro:arm_transmission prefix="${prefix}" />
+    <xacro:arm_gazebo prefix="${prefix}" />
+  </xacro:macro>
+   <xacro:arm_robot prefix=""/>
 </robot>
