Commit message: simulator work

File: Manipulator/man_gazebo/urdf/6dof/roll_z_pitch_y_pitch_y_pitch_y_pitch_z_roll_z_/roll_z_0_1pitch_y_0_7pitch_y_0_7pitch_y_0_7pitch_z_0_7roll_z_0_4.urdf.xacro (robot description, xacro)
@@ -31,5 +31,5 @@
 </xacro:macro>
   <xacro:macro name="arm_robot" params="prefix ">
-        <xacro:property name="base_length" value="0.25"/>
+        <xacro:property name="base_length" value="6.25"/>
             <!-- Inertia parameters -->
         <xacro:property name="base_mass" value="4.0" />

File: Manipulator/man_gazebo/urdf/6dof/roll_z_pitch_y_pitch_y_pitch_y_pitch_z_roll_z_/roll_z_0_1pitch_y_0_7pitch_y_0_7pitch_y_0_7pitch_z_0_7roll_z_0_7.urdf.xacro (robot description, xacro)
@@ -31,5 +31,5 @@
 </xacro:macro>
   <xacro:macro name="arm_robot" params="prefix ">
-        <xacro:property name="base_length" value="0.25"/>
+        <xacro:property name="base_length" value="6.25"/>
             <!-- Inertia parameters -->
         <xacro:property name="base_mass" value="4.0" />

File: Manipulator/man_gazebo/urdf/manip.urdf.xacro (robot description, xacro)
@@ -36,5 +36,5 @@
 	<xacro:property name="joint5_axe" value="0 1 0" />
 	<xacro:property name="joint6_axe" value="0 0 1" />
-    <xacro:property name="base_length" value="0.25" />
+    <xacro:property name="base_length" value="6.25" />
 	<xacro:property name="link1_length" value="0.15" />
 	<xacro:property name="link2_length" value="0.5" />
