Commit message: make on launch file for all launches

File: Manipulator/man_gazebo/urdf/manip.urdf.xacro (robot description, xacro)
@@ -242,5 +242,5 @@
       <parent link="${prefix}link6" />
       <child link = "${prefix}ee_link" />
-      <origin xyz="0.0 ${link6_length} 0.0" rpy="0.0 0.0 ${pi/2.0}" />
+      <origin xyz="0.0  0.0 ${link6_length}" rpy="0.0 0.0 0" />
     </joint>
 <!-- ee link -->
@@ -250,6 +250,12 @@
           <box size="0.01 0.01 0.01"/>
         </geometry>
-        <origin rpy="0 0 0" xyz="-0.01 0 0"/>
-      </collision>
+        <origin rpy="0 0 0" xyz="0 0 0.005"/>
+      </collision>
+      <visual>
+        <geometry>
+          <box size="0.01 0.01 0.01"/>
+        </geometry>
+        <origin rpy="0 0 0" xyz="0.0 0 0.005"/>
+      </visual>
     </link>
     <xacro:arm_transmission prefix="${prefix}" />

Commit message: add files

File: Manipulator/man_gazebo/urdf/manip.urdf.xacro (robot description, xacro)
@@ -1,5 +1,4 @@
 <?xml version="1.0"?>
 <robot xmlns:xacro="http://wiki.ros.org/xacro">
-asdasd
   <xacro:include filename="$(find man_gazebo)/urdf/transmission.xacro" />
   <xacro:include filename="$(find man_gazebo)/urdf/gazebo.xacro" />
@@ -62,5 +61,5 @@
     <link name="${prefix}base_link" >
       <visual>
-		<origin xyz="0 0 -0.075" rpy="0 0 0" />
+		<origin xyz="0 0 ${base_length/2}" rpy="0 0 0" />
         <geometry>
  			<cylinder radius="${base_radius}" length="${base_length}"/>
@@ -68,5 +67,5 @@
       </visual>
       <collision>
-			<origin xyz="0 0 -0.0" rpy="0 0 0" />
+			<origin xyz="0 0 ${base_length/2}" rpy="0 0 0" />
         <geometry>
 			<cylinder radius="${base_radius}" length="${base_length}"/>
@@ -74,5 +73,5 @@
       </collision>
       <xacro:cylinder_inertial radius="${base_radius}" length="${base_length}" mass="${base_mass}">
-        <origin xyz="0.0 0.0 -0.075" rpy="0 0 0" />
+        <origin xyz="0.0 0.0 ${base_length/2}" rpy="0 0 0" />
       </xacro:cylinder_inertial>
     </link>
@@ -81,5 +80,5 @@
       <parent link="${prefix}base_link" />
       <child link = "${prefix}link1" />
-      <origin xyz="0.0 0.0 0.0" rpy="0.0 0.0 0.0" />
+      <origin xyz="0.0 0.0 ${base_length/2 + link1_length/2}" rpy="0.0 0.0 0.0" />
       <axis xyz="${joint1_axe}" />
 	  <xacro:joint_limit joint_type="${joint1_type}" link_length="${link1_length}"/>

File: Manipulator/man_gazebo/urdf/manipulator.urdf.xacro (robot description, xacro)
@@ -6,5 +6,5 @@
   <xacro:include filename="$(find man_gazebo)/urdf/manip.urdf.xacro" />
   <xacro:arm_robot prefix=""/>
-  <link name="world" />
+<link name="world" />
   <joint name="world_joint" type="fixed">
     <parent link="world" />

Commit message: rearrange between computers

File: Manipulator/man_gazebo/urdf/manip.urdf.xacro (robot description, xacro)
@@ -96,9 +96,9 @@
 		 <origin xyz="0 0 ${link1_length/2}" rpy="0 0 0" />
         <geometry>
-			<cylinder radius="${link1_radius}" length="${link1_length}"/>
-        </geometry>
-      </collision>
-      <xacro:cylinder_inertial radius="${link1_length}" length="${link1_length}" mass="${link1_mass}">
-        <origin xyz="0.0 0.0 ${base_length/2}" rpy="0 0 0" />
+			<cylinder radius="${link1_radius}" length="${link1_length}"  mass="${link1_mass}"/>
+        </geometry>
+      </collision>
+      <xacro:cylinder_inertial radius="${link1_radius}" length="${link1_length}" mass="${link1_mass}">
+        <origin xyz="0.0 0.0 ${link1_length/2}" rpy="0 0 0" />
       </xacro:cylinder_inertial>
     </link>

Commit message: for virtual server check

File: Manipulator/man_gazebo/urdf/manip.urdf.xacro (robot description, xacro)
@@ -36,5 +36,5 @@
 	<xacro:property name="joint5_axe" value="0 1 0" />
 	<xacro:property name="joint6_axe" value="0 0 1" />
-    <xacro:property name="base_length" value="6.25" />
+    <xacro:property name="base_length" value="3.25" />
 	<xacro:property name="link1_length" value="0.15" />
 	<xacro:property name="link2_length" value="0.5" />
