Commit message: add roll to the last joint

File: Manipulator/man_gazebo/urdf/gazebo.xacro (robot description, xacro)
@@ -51,4 +51,7 @@
       <selfCollide>true</selfCollide>
     </gazebo>
+    <gazebo reference="camera_link">
+      <selfCollide>true</selfCollide>
+    </gazebo>
   </xacro:macro>
 </robot>

File: Manipulator/man_gazebo/urdf/manip.urdf.xacro (robot description, xacro)
@@ -270,8 +270,29 @@
       </xacro:cylinder_inertial>
     </link>
+         <!-- fake joint - the rotation about z axe of the camera is not important -->
+        <joint name="fake_joint" type="revolute">
+      <parent link="${prefix}link6" />
+      <child link = "camera_link" />
+      <origin xyz="0.0  0.0 ${link6_length}" rpy="0.0 0.0 0" />
+      <axis xyz="0 0 1"/>
+      <xacro:joint_limit joint_type="revolute" link_length="0.1"/>
+      <dynamics damping="0.0" friction="0.0"/>
+        </joint>
+    <!-- camera link -->
+        <link name="camera_link">
+          <collision>
+            <geometry>
+              <box size="0.01 0.01 0.01"/>
+            </geometry>
+            <origin rpy="0 0 0" xyz="0 0 0.005"/>
+          </collision>
+          <xacro:cylinder_inertial radius="0.01" length="0.01" mass="0.01">
+            <origin xyz="0.0 0.0 0.005" rpy="0 0 0" />
+          </xacro:cylinder_inertial>
+        </link>
     <joint name="${prefix}ee_fixed_joint" type="fixed">
-      <parent link="${prefix}link6" />
+      <parent link="${prefix}camera_link" />
       <child link = "${prefix}ee_link" />
-      <origin xyz="0.0  0.0 ${link6_length}" rpy="0.0 0.0 0" />
+      <origin xyz="0.0  0.0 0.01" rpy="0.0 0.0 0" />
     </joint>
 <!-- ee link -->
