Commit message: arrange a little

File: Manipulator/man_gazebo/urdf/3dof/transmission_3dof.xacro (robot description, xacro)
@@ -2,4 +2,13 @@
 <robot xmlns:xacro="http://wiki.ros.org/xacro">
   <xacro:macro name="arm_transmission" params="prefix">
+    <transmission name="${prefix}joint0_trans">
+      <type>transmission_interface/SimpleTransmission</type>
+      <joint name="${prefix}joint0">
+        <hardwareInterface>hardware_interface/PositionJointInterface</hardwareInterface>
+      </joint>
+      <actuator name="${prefix}joint0_motor">
+        <mechanicalReduction>1</mechanicalReduction>
+      </actuator>
+    </transmission>
     <transmission name="${prefix}joint1_trans">
       <type>transmission_interface/SimpleTransmission</type>

File: Manipulator/man_gazebo/urdf/3dof/transmission_3dof_3.xacro (robot description, xacro)
@@ -2,13 +2,4 @@
 <robot xmlns:xacro="http://wiki.ros.org/xacro">
   <xacro:macro name="arm_transmission" params="prefix">
-    <transmission name="${prefix}joint0_trans">
-      <type>transmission_interface/SimpleTransmission</type>
-      <joint name="${prefix}joint0">
-        <hardwareInterface>hardware_interface/PositionJointInterface</hardwareInterface>
-      </joint>
-      <actuator name="${prefix}joint0_motor">
-        <mechanicalReduction>1</mechanicalReduction>
-      </actuator>
-    </transmission>
     <transmission name="${prefix}joint1_trans">
       <type>transmission_interface/SimpleTransmission</type>
@@ -38,13 +29,4 @@
       </actuator>
     </transmission>
-    <transmission name="${prefix}joint4_trans">
-      <type>transmission_interface/SimpleTransmission</type>
-      <joint name="${prefix}joint4">
-        <hardwareInterface>hardware_interface/PositionJointInterface</hardwareInterface>
-      </joint>
-      <actuator name="${prefix}joint4_motor">
-        <mechanicalReduction>1</mechanicalReduction>
-      </actuator>
-    </transmission>
   </xacro:macro>
 </robot>

File: Manipulator/man_gazebo/urdf/4dof/transmission_4dof (copy).xacro (robot description, xacro)
@@ -2,13 +2,4 @@
 <robot xmlns:xacro="http://wiki.ros.org/xacro">
   <xacro:macro name="arm_transmission" params="prefix">
-    <transmission name="${prefix}joint0_trans">
-      <type>transmission_interface/SimpleTransmission</type>
-      <joint name="${prefix}joint0">
-        <hardwareInterface>hardware_interface/PositionJointInterface</hardwareInterface>
-      </joint>
-      <actuator name="${prefix}joint0_motor">
-        <mechanicalReduction>1</mechanicalReduction>
-      </actuator>
-    </transmission>
     <transmission name="${prefix}joint1_trans">
       <type>transmission_interface/SimpleTransmission</type>

File: Manipulator/man_gazebo/urdf/5dof/transmission_5dof (copy).xacro (robot description, xacro)
@@ -2,13 +2,4 @@
 <robot xmlns:xacro="http://wiki.ros.org/xacro">
   <xacro:macro name="arm_transmission" params="prefix">
-    <transmission name="${prefix}joint0_trans">
-      <type>transmission_interface/SimpleTransmission</type>
-      <joint name="${prefix}joint0">
-        <hardwareInterface>hardware_interface/PositionJointInterface</hardwareInterface>
-      </joint>
-      <actuator name="${prefix}joint0_motor">
-        <mechanicalReduction>1</mechanicalReduction>
-      </actuator>
-    </transmission>
     <transmission name="${prefix}joint1_trans">
       <type>transmission_interface/SimpleTransmission</type>
@@ -47,4 +38,13 @@
       </actuator>
     </transmission>
+   <transmission name="${prefix}joint5_trans">
+      <type>transmission_interface/SimpleTransmission</type>
+      <joint name="${prefix}joint5">
+        <hardwareInterface>hardware_interface/PositionJointInterface</hardwareInterface>
+      </joint>
+      <actuator name="${prefix}joint5_motor">
+        <mechanicalReduction>1</mechanicalReduction>
+      </actuator>
+    </transmission>
   </xacro:macro>
 </robot>

File: Manipulator/man_gazebo/urdf/5dof/transmission_5dof.xacro (robot description, xacro)
@@ -2,4 +2,13 @@
 <robot xmlns:xacro="http://wiki.ros.org/xacro">
   <xacro:macro name="arm_transmission" params="prefix">
+    <transmission name="${prefix}joint0_trans">
+      <type>transmission_interface/SimpleTransmission</type>
+      <joint name="${prefix}joint0">
+        <hardwareInterface>hardware_interface/PositionJointInterface</hardwareInterface>
+      </joint>
+      <actuator name="${prefix}joint0_motor">
+        <mechanicalReduction>1</mechanicalReduction>
+      </actuator>
+    </transmission>
     <transmission name="${prefix}joint1_trans">
       <type>transmission_interface/SimpleTransmission</type>

File: Manipulator/man_gazebo/urdf/manip.urdf.xacro (robot description, xacro)
@@ -112,5 +112,5 @@
       <parent link="${prefix}link0" />
       <child link = "${prefix}link1" />
-      <origin xyz="0.0 0.0 ${link0_length}" rpy="0.0 0 -${pi/2}" />
+      <origin xyz="0.0 0.0 ${link0_length}" rpy="${pi/2} 0 0" />
       <axis xyz="${joint1_axe}" />
 	  <xacro:joint_limit joint_type="${joint1_type}" link_length="${link1_length}"/>
