Commit message: *add roll to EE -  the orientaion of the camera isn't important

File: Manipulator/man_gazebo/urdf/3dof/manipulator.urdf.xacro (robot description, xacro)
@@ -187,8 +187,11 @@
       </xacro:cylinder_inertial>
     </link>
-    <joint name="${prefix}ee_fixed_joint" type="fixed">
+    <joint name="${prefix}ee_joint" type="revolute">
       <parent link="${prefix}link3" />
       <child link = "${prefix}ee_link" />
       <origin xyz="0.0  0.0 ${link3_length}" rpy="0.0 0.0 0" />
+      <axis xyz="0 0 1"/>
+      <xacro:joint_limit joint_type="revolute" link_length="0.01"/>
+      <dynamics damping="0.0" friction="0.0"/>
     </joint>
 <!-- ee link -->
@@ -200,4 +203,7 @@
         <origin rpy="0 0 0" xyz="0 0 0.005"/>
       </collision>
+      <xacro:cylinder_inertial radius="0.01" length="0.01" mass="0.01">
+        <origin xyz="0.0 0.0 0.005" rpy="0 0 0" />
+      </xacro:cylinder_inertial>
     </link>
     <xacro:arm_transmission prefix="${prefix}" />

File: Manipulator/man_gazebo/urdf/3dof/transmission_3dof.xacro (robot description, xacro)
@@ -38,4 +38,13 @@
       </actuator>
     </transmission>
+   <transmission name="${prefix}ee_joint_trans">
+      <type>transmission_interface/SimpleTransmission</type>
+      <joint name="${prefix}ee_joint">
+        <hardwareInterface>hardware_interface/PositionJointInterface</hardwareInterface>
+      </joint>
+      <actuator name="${prefix}ee_joint_motor">
+        <mechanicalReduction>1</mechanicalReduction>
+      </actuator>
+    </transmission>
   </xacro:macro>
 </robot>

File: Manipulator/man_gazebo/urdf/4dof/manipulator.urdf.xacro (robot description, xacro)
@@ -217,8 +217,11 @@
       </xacro:cylinder_inertial>
     </link>
-    <joint name="${prefix}ee_fixed_joint" type="fixed">
+    <joint name="${prefix}ee_joint" type="revolute">
       <parent link="${prefix}link4" />
       <child link = "${prefix}ee_link" />
       <origin xyz="0.0  0.0 ${link4_length}" rpy="0.0 0.0 0" />
+      <axis xyz="0 0 1"/>
+      <xacro:joint_limit joint_type="revolute" link_length="0.1"/>
+      <dynamics damping="0.0" friction="0.0"/>
     </joint>
 <!-- ee link -->
@@ -230,4 +233,7 @@
         <origin rpy="0 0 0" xyz="0 0 0.005"/>
       </collision>
+      <xacro:cylinder_inertial radius="0.01" length="0.01" mass="0.01">
+        <origin xyz="0.0 0.0 0.005" rpy="0 0 0" />
+      </xacro:cylinder_inertial>
     </link>
     <xacro:arm_transmission prefix="${prefix}" />

File: Manipulator/man_gazebo/urdf/4dof/transmission_4dof.xacro (robot description, xacro)
@@ -47,4 +47,13 @@
       </actuator>
     </transmission>
+   <transmission name="${prefix}ee_joint_trans">
+      <type>transmission_interface/SimpleTransmission</type>
+      <joint name="${prefix}ee_joint">
+        <hardwareInterface>hardware_interface/PositionJointInterface</hardwareInterface>
+      </joint>
+      <actuator name="${prefix}ee_joint_motor">
+        <mechanicalReduction>1</mechanicalReduction>
+      </actuator>
+    </transmission>
   </xacro:macro>
 </robot>

File: Manipulator/man_gazebo/urdf/5dof/manipulator.urdf.xacro (robot description, xacro)
@@ -85,5 +85,5 @@
         <geometry>
 			<!--<cylinder radius="${link0_radius}" length="${link0_length}"/>	  -->
-			<box size="0.3 0.6 0.4"/>
+			<box size="0.1 0.1 0.2"/>
         </geometry>
       </visual>
@@ -248,8 +248,11 @@
       </xacro:cylinder_inertial>
     </link>
-    <joint name="${prefix}ee_fixed_joint" type="fixed">
+     <joint name="${prefix}ee_joint" type="revolute">
       <parent link="${prefix}link5" />
       <child link = "${prefix}ee_link" />
       <origin xyz="0.0  0.0 ${link5_length}" rpy="0.0 0.0 0" />
+      <axis xyz="0 0 1"/>
+      <xacro:joint_limit joint_type="revolute" link_length="0.1"/>
+      <dynamics damping="0.0" friction="0.0"/>
     </joint>
 <!-- ee link -->
@@ -261,4 +264,7 @@
         <origin rpy="0 0 0" xyz="0 0 0.005"/>
       </collision>
+      <xacro:cylinder_inertial radius="0.01" length="0.01" mass="0.01">
+        <origin xyz="0.0 0.0 0.005" rpy="0 0 0" />
+      </xacro:cylinder_inertial>
     </link>
     <xacro:arm_transmission prefix="${prefix}" />

File: Manipulator/man_gazebo/urdf/5dof/transmission_5dof.xacro (robot description, xacro)
@@ -56,4 +56,13 @@
       </actuator>
     </transmission>
+   <transmission name="${prefix}ee_joint_trans">
+      <type>transmission_interface/SimpleTransmission</type>
+      <joint name="${prefix}ee_joint">
+        <hardwareInterface>hardware_interface/PositionJointInterface</hardwareInterface>
+      </joint>
+      <actuator name="${prefix}ee_joint_motor">
+        <mechanicalReduction>1</mechanicalReduction>
+      </actuator>
+    </transmission>
   </xacro:macro>
 </robot>

File: Manipulator/man_gazebo/urdf/6dof/transmission_6dof.xacro (robot description, xacro)
@@ -65,4 +65,13 @@
       </actuator>
     </transmission>
+   <transmission name="${prefix}ee_joint_trans">
+      <type>transmission_interface/SimpleTransmission</type>
+      <joint name="${prefix}ee_joint">
+        <hardwareInterface>hardware_interface/PositionJointInterface</hardwareInterface>
+      </joint>
+      <actuator name="${prefix}ee_joint_motor">
+        <mechanicalReduction>1</mechanicalReduction>
+      </actuator>
+    </transmission>
   </xacro:macro>
 </robot>

File: Manipulator/man_gazebo/urdf/manip.urdf.xacro (robot description, xacro)
@@ -270,8 +270,11 @@
       </xacro:cylinder_inertial>
     </link>
-    <joint name="${prefix}ee_fixed_joint" type="fixed">
+    <joint name="${prefix}ee_joint" type="revolute">
       <parent link="${prefix}link6" />
       <child link = "${prefix}ee_link" />
       <origin xyz="0.0  0.0 ${link6_length}" rpy="0.0 0.0 0" />
+      <axis xyz="0 0 1"/>
+      <xacro:joint_limit joint_type="revolute" link_length="0.1"/>
+      <dynamics damping="0.0" friction="0.0"/>
     </joint>
 <!-- ee link -->
@@ -283,10 +286,7 @@
         <origin rpy="0 0 0" xyz="0 0 0.005"/>
       </collision>
-      <visual>
-        <geometry>
-          <box size="0.01 0.01 0.01"/>
-        </geometry>
-        <origin rpy="0 0 0" xyz="0.0 0 0.005"/>
-      </visual>
+      <xacro:cylinder_inertial radius="0.01" length="0.01" mass="0.01">
+        <origin xyz="0.0 0.0 0.005" rpy="0 0 0" />
+      </xacro:cylinder_inertial>
     </link>
     <xacro:arm_transmission prefix="${prefix}" />

Commit message: add roll to 3-5 dofs

File: Manipulator/man_gazebo/urdf/3dof/manipulator.urdf.xacro (robot description, xacro)
@@ -187,11 +187,29 @@
       </xacro:cylinder_inertial>
     </link>
-    <joint name="${prefix}ee_joint" type="revolute">
+ <!-- fake joint - the rotation about z axe of the camera is not important -->
+        <joint name="fake_joint" type="revolute">
       <parent link="${prefix}link3" />
-      <child link = "${prefix}ee_link" />
+      <child link = "camera_link" />
       <origin xyz="0.0  0.0 ${link3_length}" rpy="0.0 0.0 0" />
       <axis xyz="0 0 1"/>
-      <xacro:joint_limit joint_type="revolute" link_length="0.01"/>
-      <dynamics damping="0.0" friction="0.0"/>
+      <xacro:joint_limit joint_type="revolute" link_length="0.1"/>
+      <dynamics damping="0.0" friction="0.0"/>
+        </joint>
+    <!-- camera link -->
+        <link name="camera_link">
+          <collision>
+            <geometry>
+              <box size="0.01 0.01 0.01"/>
+            </geometry>
+            <origin rpy="0 0 0" xyz="0 0 0.005"/>
+          </collision>
+          <xacro:cylinder_inertial radius="0.01" length="0.01" mass="0.01">
+            <origin xyz="0.0 0.0 0.005" rpy="0 0 0" />
+          </xacro:cylinder_inertial>
+        </link>
+    <joint name="${prefix}ee_fixed_joint" type="fixed">
+      <parent link="${prefix}camera_link" />
+      <child link = "${prefix}ee_link" />
+      <origin xyz="0.0  0.0 0.01" rpy="0.0 0.0 0" />
     </joint>
 <!-- ee link -->
@@ -203,8 +221,5 @@
         <origin rpy="0 0 0" xyz="0 0 0.005"/>
       </collision>
-      <xacro:cylinder_inertial radius="0.01" length="0.01" mass="0.01">
-        <origin xyz="0.0 0.0 0.005" rpy="0 0 0" />
-      </xacro:cylinder_inertial>
-    </link>
+	</link>
     <xacro:arm_transmission prefix="${prefix}" />
     <xacro:arm_gazebo prefix="${prefix}" />

File: Manipulator/man_gazebo/urdf/3dof/transmission_3dof.xacro (robot description, xacro)
@@ -38,10 +38,10 @@
       </actuator>
     </transmission>
-   <transmission name="${prefix}ee_joint_trans">
+     <transmission name="fake_joint_trans">
       <type>transmission_interface/SimpleTransmission</type>
-      <joint name="${prefix}ee_joint">
+      <joint name="fake_joint">
         <hardwareInterface>hardware_interface/PositionJointInterface</hardwareInterface>
       </joint>
-      <actuator name="${prefix}ee_joint_motor">
+      <actuator name="fake_joint_motor">
         <mechanicalReduction>1</mechanicalReduction>
       </actuator>

File: Manipulator/man_gazebo/urdf/4dof/manipulator.urdf.xacro (robot description, xacro)
@@ -217,11 +217,29 @@
       </xacro:cylinder_inertial>
     </link>
-    <joint name="${prefix}ee_joint" type="revolute">
+          <!-- fake joint - the rotation about z axe of the camera is not important -->
+        <joint name="fake_joint" type="revolute">
       <parent link="${prefix}link4" />
-      <child link = "${prefix}ee_link" />
+      <child link = "camera_link" />
       <origin xyz="0.0  0.0 ${link4_length}" rpy="0.0 0.0 0" />
       <axis xyz="0 0 1"/>
       <xacro:joint_limit joint_type="revolute" link_length="0.1"/>
       <dynamics damping="0.0" friction="0.0"/>
+        </joint>
+    <!-- camera link -->
+        <link name="camera_link">
+          <collision>
+            <geometry>
+              <box size="0.01 0.01 0.01"/>
+            </geometry>
+            <origin rpy="0 0 0" xyz="0 0 0.005"/>
+          </collision>
+          <xacro:cylinder_inertial radius="0.01" length="0.01" mass="0.01">
+            <origin xyz="0.0 0.0 0.005" rpy="0 0 0" />
+          </xacro:cylinder_inertial>
+        </link>
+    <joint name="${prefix}ee_fixed_joint" type="fixed">
+      <parent link="${prefix}camera_link" />
+      <child link = "${prefix}ee_link" />
+      <origin xyz="0.0  0.0 0.01" rpy="0.0 0.0 0" />
     </joint>
 <!-- ee link -->
@@ -233,8 +251,7 @@
         <origin rpy="0 0 0" xyz="0 0 0.005"/>
       </collision>
-      <xacro:cylinder_inertial radius="0.01" length="0.01" mass="0.01">
-        <origin xyz="0.0 0.0 0.005" rpy="0 0 0" />
-      </xacro:cylinder_inertial>
-    </link>
+	</link>
+    <xacro:arm_transmission prefix="${prefix}" />
+    <xacro:arm_gazebo prefix="${prefix}" />
     <xacro:arm_transmission prefix="${prefix}" />
     <xacro:arm_gazebo prefix="${prefix}" />

File: Manipulator/man_gazebo/urdf/4dof/transmission_4dof.xacro (robot description, xacro)
@@ -47,10 +47,10 @@
       </actuator>
     </transmission>
-   <transmission name="${prefix}ee_joint_trans">
+   <transmission name="${prefix}fake_joint_trans">
       <type>transmission_interface/SimpleTransmission</type>
-      <joint name="${prefix}ee_joint">
+      <joint name="${prefix}fake_joint">
         <hardwareInterface>hardware_interface/PositionJointInterface</hardwareInterface>
       </joint>
-      <actuator name="${prefix}ee_joint_motor">
+      <actuator name="${prefix}fake_joint_motor">
         <mechanicalReduction>1</mechanicalReduction>
       </actuator>

File: Manipulator/man_gazebo/urdf/5dof/manipulator.urdf.xacro (robot description, xacro)
@@ -248,11 +248,29 @@
       </xacro:cylinder_inertial>
     </link>
-     <joint name="${prefix}ee_joint" type="revolute">
+          <!-- fake joint - the rotation about z axe of the camera is not important -->
+        <joint name="fake_joint" type="revolute">
       <parent link="${prefix}link5" />
-      <child link = "${prefix}ee_link" />
+      <child link = "camera_link" />
       <origin xyz="0.0  0.0 ${link5_length}" rpy="0.0 0.0 0" />
       <axis xyz="0 0 1"/>
       <xacro:joint_limit joint_type="revolute" link_length="0.1"/>
       <dynamics damping="0.0" friction="0.0"/>
+        </joint>
+    <!-- camera link -->
+        <link name="camera_link">
+          <collision>
+            <geometry>
+              <box size="0.01 0.01 0.01"/>
+            </geometry>
+            <origin rpy="0 0 0" xyz="0 0 0.005"/>
+          </collision>
+          <xacro:cylinder_inertial radius="0.01" length="0.01" mass="0.01">
+            <origin xyz="0.0 0.0 0.005" rpy="0 0 0" />
+          </xacro:cylinder_inertial>
+        </link>
+    <joint name="${prefix}ee_fixed_joint" type="fixed">
+      <parent link="${prefix}camera_link" />
+      <child link = "${prefix}ee_link" />
+      <origin xyz="0.0  0.0 0.01" rpy="0.0 0.0 0" />
     </joint>
 <!-- ee link -->
@@ -264,8 +282,5 @@
         <origin rpy="0 0 0" xyz="0 0 0.005"/>
       </collision>
-      <xacro:cylinder_inertial radius="0.01" length="0.01" mass="0.01">
-        <origin xyz="0.0 0.0 0.005" rpy="0 0 0" />
-      </xacro:cylinder_inertial>
-    </link>
+	</link>
     <xacro:arm_transmission prefix="${prefix}" />
     <xacro:arm_gazebo prefix="${prefix}" />

File: Manipulator/man_gazebo/urdf/5dof/transmission_5dof.xacro (robot description, xacro)
@@ -56,10 +56,10 @@
       </actuator>
     </transmission>
-   <transmission name="${prefix}ee_joint_trans">
+   <transmission name="${prefix}fake_joint_trans">
       <type>transmission_interface/SimpleTransmission</type>
-      <joint name="${prefix}ee_joint">
+      <joint name="${prefix}fake_joint">
         <hardwareInterface>hardware_interface/PositionJointInterface</hardwareInterface>
       </joint>
-      <actuator name="${prefix}ee_joint_motor">
+      <actuator name="${prefix}fake_joint_motor">
         <mechanicalReduction>1</mechanicalReduction>
       </actuator>

Commit message: fixed bugs

File: Manipulator/man_gazebo/urdf/3dof/manipulator.urdf.xacro (robot description, xacro)
@@ -76,5 +76,5 @@
       <origin xyz="0.0 ${base_radius} ${base_length + link0_radius}" rpy="${-pi/2} 0.0 0" />
       <axis xyz="${joint0_axe}" />
-	  <xacro:joint_limit joint_type="${joint0_type}" link_length="0"/>
+	  <xacro:joint_limit joint_type="${joint0_type}" link_length="${link0_length*6}"/>
       <dynamics damping="0.0" friction="0.0"/>
     </joint>
@@ -159,10 +159,10 @@
 <xacro:property name="joint3_type" value="revolute"/>
 <xacro:property name="joint3_axe" value="0 1 0"/>
-<xacro:property name="link3_length" value="0.4"/>
+<xacro:property name="link3_length" value="0.1"/>
 <!--  joint 3	-->
     <joint name="${prefix}joint3" type="${joint3_type}">
       <parent link="${prefix}link2"/>
       <child link="${prefix}link3" />
-      <origin xyz="0 ${link2_radius+link3_radius} ${link2_length}" rpy="0 ${pi/2} 0 "/>
+      <origin xyz="0 0 ${link2_length+link3_radius}" rpy="${pi/2} 0  0 "/>
       <axis xyz="${joint3_axe}"/>
 	  <xacro:joint_limit joint_type="${joint3_type}" link_length="${link3_length}"/>

File: Manipulator/man_gazebo/urdf/4dof/manipulator.urdf.xacro (robot description, xacro)
@@ -159,5 +159,5 @@
 <xacro:property name="joint3_type" value="revolute"/>
 <xacro:property name="joint3_axe" value="0 1 0"/>
-<xacro:property name="link3_length" value="0.1"/>
+<xacro:property name="link3_length" value="0.4"/>
 <!--  joint 3	-->
     <joint name="${prefix}joint3" type="${joint3_type}">
@@ -194,5 +194,5 @@
       <parent link="${prefix}link3"/>
       <child link="${prefix}link4" />
-      <origin xyz="0 ${link3_radius+link4_radius} ${link3_length}" rpy="0 0 0 "/>
+      <origin xyz="0 0 ${link3_length+link4_radius}" rpy="${pi/2} 0 0 "/>
       <axis xyz="${joint4_axe}"/>
 	  <xacro:joint_limit joint_type="${joint4_type}" link_length="${link4_length}"/>

File: Manipulator/man_gazebo/urdf/5dof/manipulator.urdf.xacro (robot description, xacro)
@@ -51,10 +51,10 @@
         	<!--   Base Link -->
     <link name="${prefix}base_link" >
-    <!--  <visual>
+    <!---->  <visual>
 		<origin xyz="0 0 ${base_length/2}" rpy="0 0 0" />
         <geometry>
  			<cylinder radius="${base_radius}" length="${base_length}"/>
         </geometry>
-      </visual> -->
+      </visual>
       <collision>
 			<origin xyz="0 0 ${base_length/2}" rpy="0 0 0" />
@@ -74,5 +74,5 @@
       <parent link="${prefix}base_link" />
       <child link = "${prefix}link0" />
-      <origin xyz="0.0 ${base_radius} ${base_length + link0_radius}" rpy="${-pi/2} 0.0 0" />
+      <origin xyz="0.0 0 ${base_length + link0_radius+0.01}" rpy="${-pi/2} 0.0 0" />
       <axis xyz="${joint0_axe}" />
 	  <xacro:joint_limit joint_type="${joint0_type}" link_length="${link0_length*6}"/>
@@ -84,6 +84,6 @@
 		<origin xyz="0 0 ${link0_radius} " rpy="0 0 0" />
         <geometry>
-			<!--<cylinder radius="${link0_radius}" length="${link0_length}"/>	  -->
-			<box size="0.1 0.1 0.2"/>
+			<cylinder radius="${link0_radius}" length="${link0_length}"/>
+			<!--<box size="0.1 0.1 0.2"/>-->
         </geometry>
       </visual>
@@ -128,12 +128,12 @@
       </xacro:cylinder_inertial>
     </link>
-<xacro:property name="joint2_type" value="prismatic"/>
-<xacro:property name="joint2_axe" value="0 0 1"/>
-<xacro:property name="link2_length" value="0.4"/>
+<xacro:property name="joint2_type" value="revolute"/>
+<xacro:property name="joint2_axe" value="0 1 0"/>
+<xacro:property name="link2_length" value="0.5"/>
 <!--  joint 2	-->
     <joint name="${prefix}joint2" type="${joint2_type}">
       <parent link="${prefix}link1"/>
       <child link="${prefix}link2" />
-      <origin xyz="0 0 ${link1_length}" rpy="0 0 ${-pi/2} "/>
+      <origin xyz="0 ${link1_radius * 2.0} ${link1_length}" rpy="0 ${pi/2} 0 "/>
       <axis xyz="${joint2_axe}"/>
 	  <xacro:joint_limit joint_type="${joint2_type}" link_length="${link2_length}"/>
@@ -165,5 +165,5 @@
       <parent link="${prefix}link2"/>
       <child link="${prefix}link3" />
-      <origin xyz="0 ${link2_radius+link3_radius} ${link2_length}" rpy="0 ${pi/2} 0 "/>
+      <origin xyz="0 ${link2_radius+link3_radius} ${link2_length}" rpy="0 0 0 "/>
       <axis xyz="${joint3_axe}"/>
 	  <xacro:joint_limit joint_type="${joint3_type}" link_length="${link3_length}"/>

File: Manipulator/man_gazebo/urdf/5dof/transmission_5dof.xacro (robot description, xacro)
@@ -2,5 +2,5 @@
 <robot xmlns:xacro="http://wiki.ros.org/xacro">
   <xacro:macro name="arm_transmission" params="prefix">
-    <transmission name="${prefix}joint0_trans">
+ 	<transmission name="${prefix}joint0_trans">
       <type>transmission_interface/SimpleTransmission</type>
       <joint name="${prefix}joint0">
@@ -47,5 +47,5 @@
       </actuator>
     </transmission>
-   <transmission name="${prefix}joint5_trans">
+	<transmission name="${prefix}joint5_trans">
       <type>transmission_interface/SimpleTransmission</type>
       <joint name="${prefix}joint5">
@@ -56,10 +56,10 @@
       </actuator>
     </transmission>
-   <transmission name="${prefix}fake_joint_trans">
+    <transmission name="fake_joint_trans">
       <type>transmission_interface/SimpleTransmission</type>
-      <joint name="${prefix}fake_joint">
+      <joint name="fake_joint">
         <hardwareInterface>hardware_interface/PositionJointInterface</hardwareInterface>
       </joint>
-      <actuator name="${prefix}fake_joint_motor">
+      <actuator name="fake_joint_motor">
         <mechanicalReduction>1</mechanicalReduction>
       </actuator>
