Commit message: change detection points

File: Manipulator/man_gazebo/urdf/4dof/manipulator.urdf.xacro (robot description, xacro)
@@ -6,5 +6,5 @@
     <parent link="world" />
     <child link = "base_link" />
-    <origin xyz="0 -0.5 0" rpy="0.0 0.0 0.0" />
+    <origin xyz="0 -1 0" rpy="0.0 0.0 0.0" />
   </joint>
   <xacro:include filename="$(find man_gazebo)/urdf/4dof/transmission_4dof.xacro" />
@@ -76,5 +76,5 @@
       <origin xyz="0.0 ${base_radius} ${base_length + link0_radius}" rpy="${-pi/2} 0.0 0" />
       <axis xyz="${joint0_axe}" />
-	  <xacro:joint_limit joint_type="${joint0_type}" link_length="${link0_length}"/>
+	  <xacro:joint_limit joint_type="${joint0_type}" link_length="${link0_length*6}"/>
       <dynamics damping="0.0" friction="0.0"/>
     </joint>

File: Manipulator/man_gazebo/urdf/5dof/manipulator.urdf.xacro (robot description, xacro)
@@ -31,5 +31,5 @@
 </xacro:macro>
   <xacro:macro name="arm_robot" params="prefix ">
-        <xacro:property name="base_length" value="3.25"/>
+        <xacro:property name="base_length" value="0.25"/>
             <!-- Inertia parameters -->
         <xacro:property name="base_mass" value="1.0" />

File: Manipulator/man_gazebo/urdf/manip.urdf.xacro (robot description, xacro)
@@ -39,5 +39,5 @@
 	<xacro:property name="joint6_axe" value="0 0 1" />
 	<xacro:property name="link0_length" value="0.25" />
-    <xacro:property name="base_length"  value="3.25" />
+    <xacro:property name="base_length"  value="0.25" />
 	<xacro:property name="link1_length" value="0.25" />
 	<xacro:property name="link2_length" value="0.5" />
