Commit message: add loggong launch

File: Manipulator/man_gazebo/urdf/5dof/manipulator.urdf.xacro (robot description, xacro)
@@ -31,5 +31,5 @@
 </xacro:macro>
   <xacro:macro name="arm_robot" params="prefix ">
-        <xacro:property name="base_length" value="0.25"/>
+        <xacro:property name="base_length" value="3.25"/>
             <!-- Inertia parameters -->
         <xacro:property name="base_mass" value="1.0" />
